File: hardware/sam7x-nrf.sch (EAGLE design)
At the start: 88 parts, among them CN2 RJ45-8PTH, IC1 AT91SAM7X256-AU, J2 J0026, Q1 BSS???, U1 KSZ8081RNA, U2 NRF24L01SMD, U3 USD-SOCKETUSD, U4 MICXXXX, U5 MAX3051, Y1 18.432, Y2 16M, Y3 25MHz

Commit message: rc
Parts:
- removed BOX1: HAMMOND-BOX-XXA, hammond:HAMMOND-BOX-XXA
- removed C10: 10n, rcl:C-EUC0603
- removed C22, C23, C24, C25, C26, C27, C28, C32, C38: .1u, rcl:C-EUC0603
- removed CN2: RJ45-8PTH, sparkfun:RJ45-8PTH
- removed IC1: AT91SAM7X256-AU, balto:AT91SAM7X256-AU
- removed JP4: (no value), pinhead:PINHD-1X4
- removed JP7: (no value), pinhead:PINHD-1X2
- removed LED2: (no value), led:LEDCHIPLED_0805
- removed Q1: BSS???, SparkFun-DiscreteSemi:MOSFET-PCHANNELSMD
- removed R10, R14: 330k, rcl:R-EU_R0603
- removed R12: 330, rcl:R-EU_R0603
- removed R15: 1k5, rcl:R-EU_R0603
- removed U3: USD-SOCKETUSD, SparkFun-Connectors:USD-SOCKETUSD
- added C40: 1u, rcl:C-EUC0603
- added J3: RJ45-8PTH, balto:RJ45-8PTH
- added JP1: (no value), SparkFun-Connectors:M04PTH
- added SJ1: (no value), SparkFun-Passives:SOLDERJUMPER_2WAYS
- added U6: STM32F107XX, balto:STM32F107XX
- C29, C30: value 10p -> 16p
- C9: value 1n -> .1u
- R16, R35: device rcl:R-EU_R0603 -> rcl:R-EU_R0805
- R17: value 27 -> 10k
- R7, R8: value 27 -> 22
- R9: value 1k5 -> 10k
- S3: device sparkfun:SWITCH-MOMENTARY-2PTH -> sparkfun:SWITCH-MOMENTARY-2SMD
- U$5: value INVERTED_F_ANTENNA+5 -> INVERTED_F_ANTENNA-2; device antenna:INVERTED_F_ANTENNA+5 -> antenna:INVERTED_F_ANTENNA-2
- U4: value MICXXXX -> MIC5301
- Y1: value 18.432 -> 8MHz
Connections:
- removed net 1.8V: C23.1, C24.1, C25.1, C26.1, C27.1, C28.1, IC1.VDDCORE@1, IC1.VDDCORE@2, IC1.VDDCORE@3, IC1.VDDCORE@4, IC1.VDDOUT@1, IC1.VDDPLL
- removed net AVDREF: C38.1, IC1.ADVREF, R17.2
- removed net DBGUART_RX: IC1.PA27/DRXD/PCK3, JP4.2, R4.1
- removed net DBGUART_TX: IC1.PA28/DTXD, JP4.3
- removed net ERASE: IC1.ERASE, JP2.2
- removed net LED_C: IC1.AD2/PWM2/PCK1/PB29, LED2.A
- removed net LED_D: IC1.AD3/PWM3/PCK2/PB30, LED1.A
- removed net N$18: C29.1, IC1.XOUT, Y1.1
- removed net N$23: C10.1, R9.1
- removed net N$28: Q1.D, R15.2
- removed net N$5: LED2.C, R12.2
- removed net PHY_IRQ: U1.INTRP
- removed net PLLRC: C9.1, IC1.PLLRC, R9.2
- removed net SD_CS: U3.CS
- removed net SD_DETECT: U3.SHIELD@1
- removed net SD_DI: U3.DI
- removed net SD_DO: U3.DO
- removed net SD_SCK: U3.SCK
- removed net USB_PUEN: Q1.G
- removed net VIN_USB: U$4.VBUS, U4.EN, U4.IN
- new net BOOT0: R9.2, U6.BOOT0
- new net BOOT1: R17.2, U6.PB2
- new net ETH_IRQ: U1.INTRP, U6.PA5
- new net LED_PPS: R11.2, U6.PB5
- new net STM_OSCIN: C29.1, U6.OSC_IN, Y1.2
- new net STM_OSCOUT: C30.1, U6.OSC_OUT, Y1.1
- new net UART_RX: JP1.2, R4.1, U6.PB7
- new net UART_TX: JP1.3, U6.PB6
- new net USB_ID: U$4.ID, U6.PA10
- new net USB_VBUS: C40.1, U$4.VBUS, U4.EN, U4.IN, U6.PA9
- net CANH: now also J3.1; no longer CN2.1
- net CANL: now also J3.2, JP2.1; no longer CN2.2, JP7.2
- net CAN_RX: now also U6.PB8; no longer IC1.PA19/CANRX
- net CAN_SHDN: now also U6.PB14
- net CAN_TX: now also U6.PB9; no longer IC1.PA20/CANTX
- net ETH_RST: now also U6.PA4
- net GND: now also C40.2, JP1.4, LED1.C, LED3.C, LED5.C, R17.1, SJ1.1, U6.VSS@18, U6.VSS@31, U6.VSS@47, U6.VSS@63, U6.VSSA@12; no longer C10.2, C22.2, C23.2, C24.2, C25.2, C26.2, C27.2, C28.2, C32.2, C38.2, IC1.GND@1, IC1.GND@2, IC1.GND@3, IC1.GND@4, IC1.GND@5, IC1.GND@6, IC1.GND@7, IC1.JTAGSEL, JP4.4, R10.1, R11.1, R12.1, R13.1, R14.1, R6.1, U3.GND, U3.SHIELD@2, U3.SHIELD@3, U3.SHIELD@4
- net LED_A: now also R6.2, U6.PC14-OSC32_IN; no longer IC1.AD0/PWM0/TIOA2/PB27, LED5.A
- net LED_B: now also R13.2, U6.PC15_OSC32_OUT; no longer IC1.AD1/PWM1/TIOB2/PB28, LED3.A
- net MDC: now also U6.PC1; no longer IC1.EMDC/PB8
- net MDIO: now also U6.PA2; no longer IC1.EMDIO/PB9
- net N$12: now also LED5.A, R6.1; no longer LED5.C, R6.2
- net N$17: now also R9.1, SJ1.2; no longer C30.1, IC1.XIN/PGMCK, Y1.2
- net N$2: now also LED1.A, R11.1; no longer LED1.C, R11.2
- net N$22: no longer R10.2
- net N$26: no longer R14.2, R15.1
- net N$27: now also JP2.2; no longer JP7.1
- net N$29: now also J3.7, J3.8; no longer CN2.7, CN2.8
- net N$6: now also LED3.A, R13.1; no longer LED3.C, R13.2
- net RESET: now also C9.1, U6.NRST; no longer IC1.NRST
- net RF_CE: now also U6.PB4
- net RF_CSN: now also U6.PB3
- net RF_IRQ: now also U6.PA15
- net RF_MISO: now also U6.PC11
- net RF_MOSI: now also U6.PC12
- net RF_SCK: now also U6.PC10
- net RMII_CLK: now also U6.PA1; no longer IC1.PCK0/EREFCK/ETXCKP/B0
- net RMII_CRSDV: now also U6.PA7; no longer IC1.ERXDV/ECRSDV/PB15
- net RMII_RXD0: now also U6.PC4; no longer IC1.ERX0/PB5
- net RMII_RXD1: now also U6.PC5; no longer IC1.ERX1/PB6
- net RMII_RXER: now also U6.PA6; no longer IC1.ERXER/PB7
- net RMII_TXD0: now also U6.PB12; no longer IC1.ETX0/PB2
- net RMII_TXD1: now also U6.PB13; no longer IC1.ETX1/PB3
- net RMII_TXEN: now also U6.PB11; no longer IC1.ETXEN/PB1
- net USB_D+: now also U6.PA12; no longer IC1.DDP
- net USB_D-: now also U6.PA11; no longer IC1.DDM
- net VCC: now also JP1.1, SJ1.3, U6.VBAT, U6.VDD@19, U6.VDD@32, U6.VDD@48, U6.VDD@64, U6.VDDA@13; no longer C22.1, C32.1, IC1.VDDFLASH, IC1.VDDIN@1, IC1.VDDIO@1, IC1.VDDIO@2, IC1.VDDIO@3, IC1.VDDIO@4, IC1.VDDIO@5, JP2.1, JP4.1, Q1.S, R17.1, U3.VCC
Other:
- note added: "Alternative: 25MHz"
- note added: "CAN1"
- note added: "ETH"
- note added: "GPIO"
- note added: "SPI3"
- note added: "UART1"
- note removed: "uSD"
- moved on the sheet: C17, C18, C19, C20, C21, C29, C30, C39, C6, C8, C9, JP2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

Commit message: rc
Connections:
- net CAN_SHDN: now also U6.PA8; no longer U6.PB14
Changed lines of the file:
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@@
 25MHz</text>
 <text x="15.24" y="147.32" size="1.778" layer="97" rot="MR0">GPIO</text>
-<text x="96.52" y="106.68" size="1.778" layer="97">GPIO</text>
+<text x="96.52" y="165.1" size="1.778" layer="97">GPIO</text>
 </plain>
 <instances>
@@
 </segment>
 <segment>
-<pinref part="U6" gate="G$1" pin="PB14"/>
-<wire x1="76.2" y1="106.68" x2="93.98" y2="106.68" width="0.1524" layer="91"/>
-<label x="93.98" y="106.68" size="1.778" layer="95" rot="MR0"/>
+<label x="93.98" y="165.1" size="1.778" layer="95" rot="MR0"/>
+<wire x1="76.2" y1="165.1" x2="93.98" y2="165.1" width="0.1524" layer="91"/>
+<pinref part="U6" gate="G$1" pin="PA8"/>
 </segment>
 </net>
@@
 </sheet>
 </sheets>
+<errors>
+</errors>
 </schematic>
 </drawing>
