File: hardware/nrf-ethernet.brd (EAGLE design)
At the start: 74 x 34 mm, 71 parts, among them J2 J0026, J3 RJ45-8PTH, U1 KSZ8081RNA, U2 NRF24L01SMD, U4 MIC5301, U5 MAX3051, U6 STM32F107XX, Y1 8MHz, Y2 16M, Y3 25MHz

Commit message: rc
Parts:
- moved C29 0.41 mm to (42.7, 31.3)
- moved C30 0.41 mm to (39.8, 31.3)
- moved Y1 0.41 mm to (41.2, 31.3)
Routing:
- net GND: track 43.1 -> 56.9 mm
- net VCC: track 230.4 -> 229.8 mm, vias 12 -> 11
Changed lines of the file:
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@@
 <setting verticaltext="up"/>
 </settings>
-<grid distance="8" unitdist="mil" unit="mil" style="lines" multiple="1" display="yes" altdistance="2" altunitdist="mil" altunit="mil"/>
+<grid distance="8" unitdist="mil" unit="mil" style="lines" multiple="1" display="no" altdistance="2" altunitdist="mil" altunit="mil"/>
 <layers>
 <layer number="1" name="Top" color="4" fill="1" visible="yes" active="yes"/>
@@
 <dimension x1="6.2992" y1="0" x2="53.4416" y2="-3.048" x3="-2.4384" y3="-1.524" textsize="1.778" layer="20" dtype="vertical"/>
 <rectangle x1="54.2544" y1="15.0368" x2="55.88" y2="16.6624" layer="29"/>
-<dimension x1="58.5216" y1="3.8608" x2="66.6496" y2="3.4544" x3="62.5856" y3="-13.208" textsize="1.778" layer="20" dtype="horizontal"/>
 </plain>
 <attributes>
@@
 <element name="LED3" library="led" package="CHIPLED_0805" value="" x="49.3776" y="32.9184" rot="R90"/>
 <element name="S3" library="sparkfun" package="TACTILE_SWITCH_SMD" value="SWITCH" x="25.6032" y="30.8864" rot="R180"/>
-<element name="Y1" library="sparkfun" package="CRYSTAL-SMD-5X3" value="8MHz" x="41.2496" y="31.6992"/>
+<element name="Y1" library="sparkfun" package="CRYSTAL-SMD-5X3" value="8MHz" x="41.2496" y="31.2928"/>
 <element name="U5" library="balto" package="SO08" value="MAX3051" x="31.496" y="5.08" rot="MR180"/>
 <element name="R35" library="rcl" package="R0805" value="120" x="24.9936" y="13.8176" rot="MR90"/>
@@
 <element name="C8" library="rcl" package="C0603" value=".1u" x="41.8592" y="4.064" rot="MR225"/>
 <element name="U4" library="SparkFun-PowerIC" package="SOT23-5" value="MIC5301" x="41.656" y="8.128" rot="MR180"/>
-<element name="C29" library="rcl" package="C0603" value="16p" x="42.672" y="31.6992" rot="MR270"/>
-<element name="C30" library="rcl" package="C0603" value="16p" x="39.8272" y="31.6992" rot="MR90"/>
+<element name="C29" library="rcl" package="C0603" value="16p" x="42.672" y="31.2928" rot="MR270"/>
+<element name="C30" library="rcl" package="C0603" value="16p" x="39.8272" y="31.2928" rot="MR90"/>
 <element name="C6" library="rcl" package="C0603" value=".1u" x="30.8864" y="26.0096" rot="R180"/>
 <element name="C17" library="rcl" package="C0603" value=".1u" x="36.9824" y="31.496" rot="R90"/>
@@
 <wire x1="18.0848" y1="26.6192" x2="18.288" y2="26.416" width="0.2032" layer="1"/>
 <wire x1="14.4272" y1="26.6192" x2="14.224" y2="26.416" width="0.2032" layer="1"/>
+<wire x1="37.7952" y1="33.3248" x2="44.704" y2="33.3248" width="0.2032" layer="1"/>
+<wire x1="44.704" y1="33.3248" x2="37.7952" y2="33.3248" width="0.2032" layer="16"/>
 </signal>
 <signal name="TX+">
@@
 <wire x1="7.3152" y1="26.0096" x2="7.3152" y2="28.8544" width="0.2032" layer="1"/>
 <wire x1="7.3152" y1="28.8544" x2="7.7216" y2="29.2608" width="0.2032" layer="1"/>
-<wire x1="7.7216" y1="29.2608" x2="10.16" y2="29.2608" width="0.2032" layer="1"/>
-<wire x1="10.16" y1="29.2608" x2="10.9728" y2="28.448" width="0.2032" layer="1"/>
-<wire x1="10.9728" y1="28.448" x2="13.6144" y2="28.448" width="0.2032" layer="1"/>
+<wire x1="7.7216" y1="29.2608" x2="10.3632" y2="29.2608" width="0.2032" layer="1"/>
+<wire x1="10.3632" y1="29.2608" x2="11.176" y2="28.448" width="0.2032" layer="1"/>
+<wire x1="11.176" y1="28.448" x2="13.6144" y2="28.448" width="0.2032" layer="1"/>
 <wire x1="13.6144" y1="28.448" x2="14.224" y2="27.8384" width="0.2032" layer="1"/>
 <wire x1="14.224" y1="27.8384" x2="20.32" y2="27.8384" width="0.2032" layer="1"/>
@@
 <wire x1="34.544" y1="1.016" x2="34.544" y2="5.4492" width="0.4064" layer="16"/>
 <wire x1="32.131" y1="6.643" x2="32.131" y2="7.6962" width="0.4064" layer="16"/>
-<wire x1="42.9676" y1="28.7116" x2="43.7484" y2="28.7116" width="0.254" layer="1"/>
-<wire x1="43.7484" y1="28.7116" x2="44.704" y2="29.6672" width="0.254" layer="1"/>
-<wire x1="44.704" y1="29.6672" x2="45.6828" y2="29.6672" width="0.254" layer="1"/>
+<wire x1="42.9676" y1="28.7116" x2="43.9516" y2="28.7116" width="0.254" layer="1"/>
+<wire x1="43.9516" y1="28.7116" x2="44.9072" y2="29.6672" width="0.254" layer="1"/>
+<wire x1="44.9072" y1="29.6672" x2="45.6828" y2="29.6672" width="0.254" layer="1"/>
 <wire x1="44.9676" y1="26.7116" x2="44.9676" y2="27.7328" width="0.254" layer="1"/>
 <wire x1="44.9676" y1="27.7328" x2="45.6828" y2="28.448" width="0.254" layer="1"/>
@@
 <wire x1="35.7632" y1="31.0896" x2="35.1908" y2="31.0896" width="0.254" layer="1"/>
 <wire x1="35.1908" y1="31.0896" x2="34.544" y2="31.7364" width="0.254" layer="1"/>
-<via x="45.72" y="30.8864" extent="1-16" drill="0.508"/>
-<wire x1="45.72" y1="30.8864" x2="45.72" y2="29.7044" width="0.254" layer="1"/>
 <wire x1="45.72" y1="29.7044" x2="45.6828" y2="29.6672" width="0.254" layer="1"/>
 <wire x1="45.6828" y1="28.448" x2="45.6828" y2="29.6672" width="0.254" layer="1"/>
@@
 <wire x1="53.0352" y1="29.6672" x2="54.864" y2="29.6672" width="0.4064" layer="16"/>
 <wire x1="42.4688" y1="23.5712" x2="45.72" y2="26.8224" width="0.4064" layer="16"/>
-<wire x1="45.72" y1="30.8864" x2="48.9712" y2="30.8864" width="0.4064" layer="1"/>
+<wire x1="46.902" y1="30.8864" x2="48.9712" y2="30.8864" width="0.4064" layer="1"/>
 <wire x1="48.9712" y1="30.8864" x2="50.1904" y2="29.6672" width="0.4064" layer="1"/>
 <wire x1="50.1904" y1="29.6672" x2="50.1904" y2="26.8224" width="0.4064" layer="1"/>
@@
 <wire x1="40.2336" y1="23.5712" x2="39.8272" y2="23.1648" width="0.4064" layer="16"/>
 <wire x1="50.1904" y1="26.8224" x2="55.0672" y2="21.9456" width="0.4064" layer="16"/>
+<wire x1="46.902" y1="30.8864" x2="45.6828" y2="29.6672" width="0.4064" layer="1"/>
 </signal>
 <signal name="N$3">
@@
 <contactref element="C29" pad="1"/>
 <contactref element="Y1" pad="3"/>
-<via x="41.4528" y="32.9184" extent="1-16" drill="0.508"/>
-<wire x1="40.9676" y1="28.7116" x2="40.9676" y2="29.9948" width="0.254" layer="1"/>
-<wire x1="40.9676" y1="29.9948" x2="41.656" y2="30.6832" width="0.254" layer="1"/>
-<wire x1="41.656" y1="30.6832" x2="41.656" y2="31.6992" width="0.254" layer="1"/>
-<wire x1="41.656" y1="31.6992" x2="42.806" y2="32.8492" width="0.254" layer="1"/>
-<wire x1="42.806" y1="32.8492" x2="43.0996" y2="32.8492" width="0.254" layer="1"/>
-<wire x1="43.0996" y1="32.8492" x2="43.0304" y2="32.9184" width="0.254" layer="1"/>
-<wire x1="43.0304" y1="32.9184" x2="41.4528" y2="32.9184" width="0.254" layer="1"/>
-<wire x1="42.672" y1="32.5492" x2="41.822" y2="32.5492" width="0.254" layer="16"/>
-<wire x1="41.822" y1="32.5492" x2="41.4528" y2="32.9184" width="0.254" layer="16"/>
+<via x="41.4528" y="32.512" extent="1-16" drill="0.508"/>
+<wire x1="40.9676" y1="28.7116" x2="40.9676" y2="29.5884" width="0.254" layer="1"/>
+<wire x1="40.9676" y1="29.5884" x2="41.656" y2="30.2768" width="0.254" layer="1"/>
+<wire x1="41.656" y1="30.2768" x2="41.656" y2="31.2928" width="0.254" layer="1"/>
+<wire x1="41.656" y1="31.2928" x2="42.806" y2="32.4428" width="0.254" layer="1"/>
+<wire x1="42.806" y1="32.4428" x2="43.0996" y2="32.4428" width="0.254" layer="1"/>
+<wire x1="43.0996" y1="32.4428" x2="43.0304" y2="32.512" width="0.254" layer="1"/>
+<wire x1="43.0304" y1="32.512" x2="41.4528" y2="32.512" width="0.254" layer="1"/>
+<wire x1="42.672" y1="32.1428" x2="41.822" y2="32.1428" width="0.254" layer="16"/>
+<wire x1="41.822" y1="32.1428" x2="41.4528" y2="32.512" width="0.254" layer="16"/>
 </signal>
 <signal name="STM_OSCOUT">
@@
 <contactref element="C30" pad="1"/>
 <contactref element="Y1" pad="1"/>
-<via x="40.8432" y="31.0896" extent="1-16" drill="0.508"/>
-<wire x1="39.8272" y1="30.8492" x2="40.6028" y2="30.8492" width="0.254" layer="16"/>
-<wire x1="40.6028" y1="30.8492" x2="40.8432" y2="31.0896" width="0.254" layer="16"/>
-<wire x1="39.3996" y1="30.5492" x2="40.506" y2="30.5492" width="0.254" layer="1"/>
-<wire x1="40.506" y1="30.5492" x2="40.8432" y2="30.8864" width="0.254" layer="1"/>
-<wire x1="40.8432" y1="30.8864" x2="40.8432" y2="31.0896" width="0.254" layer="1"/>
-<wire x1="40.4676" y1="28.7116" x2="40.4676" y2="29.8396" width="0.254" layer="1"/>
-<wire x1="40.4676" y1="29.8396" x2="39.758" y2="30.5492" width="0.254" layer="1"/>
-<wire x1="39.758" y1="30.5492" x2="39.3996" y2="30.5492" width="0.254" layer="1"/>
+<via x="40.8432" y="30.6832" extent="1-16" drill="0.508"/>
+<wire x1="39.8272" y1="30.4428" x2="40.6028" y2="30.4428" width="0.254" layer="16"/>
+<wire x1="40.6028" y1="30.4428" x2="40.8432" y2="30.6832" width="0.254" layer="16"/>
+<wire x1="39.3996" y1="30.1428" x2="40.506" y2="30.1428" width="0.254" layer="1"/>
+<wire x1="40.506" y1="30.1428" x2="40.8432" y2="30.48" width="0.254" layer="1"/>
+<wire x1="40.8432" y1="30.48" x2="40.8432" y2="30.6832" width="0.254" layer="1"/>
+<wire x1="40.4676" y1="28.7116" x2="40.4676" y2="29.4332" width="0.254" layer="1"/>
+<wire x1="40.4676" y1="29.4332" x2="39.758" y2="30.1428" width="0.254" layer="1"/>
+<wire x1="39.758" y1="30.1428" x2="39.3996" y2="30.1428" width="0.254" layer="1"/>
 </signal>
 <signal name="BOOT0">
