File: hardware/nrf-ethernet.brd (EAGLE design)
At the start: 74 x 34 mm, 71 parts, among them J2 J0026, J3 RJ45-8PTH, U1 KSZ8081RNA, U2 NRF24L01SMD, U4 MIC5301, U5 MAX3051, U6 STM32F107XX, Y1 8MHz, Y2 16M, Y3 25MHz

Commit message: rc
Parts:
- moved LED5 3.86 mm to (52.2, 32.9)
- moved R6 3.86 mm to (52.2, 32.9)
- moved LED3 1.83 mm to (47.5, 32.9)
- moved R13 1.83 mm to (47.5, 32.9)
Routing:
- net LED_A: track 20.6 -> 16.7 mm
- net LED_B: track 14.2 -> 12.4 mm
Changed lines of the file:
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@@
 <element name="J2" library="micrel" package="PJ-J0" value="J0026" x="14.6304" y="8.128" rot="R180"/>
 <element name="LED1" library="led" package="CHIPLED_0805" value="" x="62.7888" y="32.9184" rot="R90"/>
-<element name="LED3" library="led" package="CHIPLED_0805" value="" x="49.3776" y="32.9184" rot="R90"/>
+<element name="LED3" library="led" package="CHIPLED_0805" value="" x="47.5488" y="32.9184" rot="R90"/>
 <element name="S3" library="sparkfun" package="TACTILE_SWITCH_SMD" value="SWITCH" x="25.6032" y="30.8864" rot="R180"/>
 <element name="Y1" library="sparkfun" package="CRYSTAL-SMD-5X3" value="8MHz" x="41.2496" y="31.2928"/>
@@
 <element name="R4" library="rcl" package="R0603" value="10k" x="56.2864" y="27.6352" rot="R180"/>
 <element name="R11" library="rcl" package="R0603" value="330" x="62.7888" y="32.9184" rot="MR0"/>
-<element name="R13" library="rcl" package="R0603" value="330" x="49.3776" y="32.9184" rot="MR0"/>
+<element name="R13" library="rcl" package="R0603" value="330" x="47.5488" y="32.9184" rot="MR0"/>
 <element name="U$4" library="SparkFun-Connectors" package="USB-MINIB" value="USB-MINIB-5PIN" x="45.5168" y="4.6736" rot="R90"/>
 <element name="C11" library="rcl" package="C0603" value="1p5" x="63.1952" y="16.4592"/>
@@
 <element name="R5" library="rcl" package="R0603" value="330" x="2.4384" y="30.6832" rot="R90"/>
 <element name="C37" library="rcl" package="C0603" value=".1u" x="15.4432" y="11.5824" rot="MR270"/>
-<element name="LED5" library="led" package="CHIPLED_0805" value="" x="56.0832" y="32.9184" rot="R90"/>
-<element name="R6" library="rcl" package="R0603" value="330" x="56.0832" y="32.9184" rot="MR0"/>
+<element name="LED5" library="led" package="CHIPLED_0805" value="" x="52.2224" y="32.9184" rot="R90"/>
+<element name="R6" library="rcl" package="R0603" value="330" x="52.2224" y="32.9184" rot="MR0"/>
 <element name="R7" library="rcl" package="R0603" value="22" x="44.3992" y="10.7696" rot="R90"/>
 <element name="R8" library="rcl" package="R0603" value="22" x="45.8216" y="10.7696" rot="R90"/>
@@
 <contactref element="LED3" pad="A"/>
 <contactref element="R13" pad="1"/>
-<wire x1="50.4276" y1="32.9184" x2="51.6128" y2="32.9184" width="0.254" layer="1"/>
-<via x="51.6128" y="32.9184" extent="1-16" drill="0.508"/>
-<wire x1="51.6128" y1="32.9184" x2="50.2276" y2="32.9184" width="0.254" layer="16"/>
+<wire x1="48.5988" y1="32.9184" x2="49.784" y2="32.9184" width="0.254" layer="1"/>
+<via x="49.784" y="32.9184" extent="1-16" drill="0.508"/>
+<wire x1="49.784" y1="32.9184" x2="48.3988" y2="32.9184" width="0.254" layer="16"/>
 </signal>
 <signal name="N$12">
 <contactref element="LED5" pad="A"/>
 <contactref element="R6" pad="1"/>
-<wire x1="56.9332" y1="32.9184" x2="58.3184" y2="32.9184" width="0.254" layer="16"/>
-<via x="58.3184" y="32.9184" extent="1-16" drill="0.508"/>
-<wire x1="58.3184" y1="32.9184" x2="57.1332" y2="32.9184" width="0.254" layer="1"/>
+<wire x1="53.0724" y1="32.9184" x2="54.4576" y2="32.9184" width="0.254" layer="16"/>
+<via x="54.4576" y="32.9184" extent="1-16" drill="0.508"/>
+<wire x1="54.4576" y1="32.9184" x2="53.2724" y2="32.9184" width="0.254" layer="1"/>
 </signal>
 <signal name="LED_B">
 <contactref element="R13" pad="2"/>
 <contactref element="U6" pad="4"/>
-<wire x1="48.5276" y1="32.9184" x2="45.9232" y2="32.9184" width="0.2032" layer="16"/>
+<wire x1="46.6988" y1="32.9184" x2="45.9232" y2="32.9184" width="0.2032" layer="16"/>
 <wire x1="45.9232" y1="32.9184" x2="44.2976" y2="31.2928" width="0.2032" layer="16"/>
 <wire x1="44.2976" y1="31.2928" x2="44.2976" y2="28.6512" width="0.2032" layer="16"/>
@@
 <contactref element="R6" pad="2"/>
 <contactref element="U6" pad="3"/>
-<wire x1="55.2332" y1="32.9184" x2="54.2172" y2="31.9024" width="0.2032" layer="16"/>
-<wire x1="54.2172" y1="31.9024" x2="45.5168" y2="31.9024" width="0.2032" layer="16"/>
+<wire x1="51.3724" y1="32.9184" x2="50.3564" y2="31.9024" width="0.2032" layer="16"/>
+<wire x1="50.3564" y1="31.9024" x2="45.5168" y2="31.9024" width="0.2032" layer="16"/>
 <wire x1="45.5168" y1="31.9024" x2="44.704" y2="31.0896" width="0.2032" layer="16"/>
 <wire x1="44.704" y1="31.0896" x2="44.704" y2="28.448" width="0.2032" layer="16"/>

Commit message: rc
Parts:
- moved LED4 2.64 mm to (7.52, 32.9)
- moved R5 0.41 mm to (2.44, 31.1)
Routing:
- net VCC: track 229.8 -> 235.2 mm
- net N$1: track 1.96 -> 4.44 mm
Changed lines of the file:
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@@
 <setting verticaltext="up"/>
 </settings>
-<grid distance="8" unitdist="mil" unit="mil" style="lines" multiple="1" display="no" altdistance="2" altunitdist="mil" altunit="mil"/>
+<grid distance="8" unitdist="mil" unit="mil" style="lines" multiple="1" display="yes" altdistance="2" altunitdist="mil" altunit="mil"/>
 <layers>
 <layer number="1" name="Top" color="4" fill="1" visible="yes" active="yes"/>
@@
 <element name="C16" library="rcl" package="C0603" value="18p" x="17.8816" y="21.5392" rot="R90"/>
 <element name="C31" library="rcl" package="C0603" value="18p" x="16.4592" y="25.8064"/>
-<element name="LED4" library="led" package="CHIPLED_0805" value="" x="4.8768" y="32.9184" rot="R90"/>
-<element name="R5" library="rcl" package="R0603" value="330" x="2.4384" y="30.6832" rot="R90"/>
+<element name="LED4" library="led" package="CHIPLED_0805" value="" x="7.5184" y="32.9184" rot="R90"/>
+<element name="R5" library="rcl" package="R0603" value="330" x="2.4384" y="31.0896" rot="R90"/>
 <element name="C37" library="rcl" package="C0603" value=".1u" x="15.4432" y="11.5824" rot="MR270"/>
 <element name="LED5" library="led" package="CHIPLED_0805" value="" x="52.2224" y="32.9184" rot="R90"/>
@@
 <wire x1="0.6096" y1="26.8224" x2="1.016" y2="27.2288" width="0.4064" layer="16"/>
 <wire x1="1.016" y1="27.2288" x2="0.6096" y2="27.6352" width="0.4064" layer="16"/>
-<wire x1="0.6096" y1="27.6352" x2="0.6096" y2="31.0896" width="0.4064" layer="16"/>
+<wire x1="0.6096" y1="27.6352" x2="0.6096" y2="32.512" width="0.4064" layer="16"/>
 <wire x1="6.9088" y1="4.8768" x2="4.8768" y2="6.9088" width="0.4064" layer="16"/>
 <wire x1="4.8768" y1="6.9088" x2="1.8288" y2="6.9088" width="0.4064" layer="16"/>
@@
 <wire x1="1.016" y1="17.0688" x2="0.6096" y2="17.4752" width="0.4064" layer="16"/>
 <wire x1="3.4544" y1="17.0688" x2="1.016" y2="17.0688" width="0.4064" layer="16"/>
-<wire x1="5.9268" y1="32.9184" x2="5.9268" y2="31.53" width="0.4064" layer="1"/>
-<wire x1="5.9268" y1="31.53" x2="5.8928" y2="31.496" width="0.4064" layer="1"/>
-<via x="5.8928" y="31.496" extent="1-16" drill="0.508"/>
-<wire x1="0.6096" y1="31.0896" x2="1.016" y2="31.496" width="0.4064" layer="16"/>
-<wire x1="1.016" y1="31.496" x2="5.8928" y2="31.496" width="0.4064" layer="16"/>
+<via x="9.9568" y="32.9184" extent="1-16" drill="0.508"/>
+<wire x1="0.6096" y1="32.512" x2="1.016" y2="32.9184" width="0.4064" layer="16"/>
+<wire x1="1.016" y1="32.9184" x2="9.9568" y2="32.9184" width="0.4064" layer="16"/>
 <wire x1="9.5504" y1="27.2288" x2="1.016" y2="27.2288" width="0.4064" layer="16"/>
 <wire x1="34.544" y1="1.016" x2="34.544" y2="5.4492" width="0.4064" layer="16"/>
@@
 <wire x1="50.1904" y1="26.8224" x2="55.0672" y2="21.9456" width="0.4064" layer="16"/>
 <wire x1="46.902" y1="30.8864" x2="45.6828" y2="29.6672" width="0.4064" layer="1"/>
+<wire x1="9.9568" y1="32.9184" x2="8.5684" y2="32.9184" width="0.4064" layer="1"/>
 </signal>
 <signal name="N$3">
@@
 <wire x1="1.8288" y1="24.7904" x2="1.8288" y2="27.2288" width="0.2032" layer="1"/>
 <wire x1="1.8288" y1="27.2288" x2="2.4384" y2="27.8384" width="0.2032" layer="1"/>
-<wire x1="2.4384" y1="27.8384" x2="2.4384" y2="29.8332" width="0.2032" layer="1"/>
+<wire x1="2.4384" y1="27.8384" x2="2.4384" y2="30.2396" width="0.2032" layer="1"/>
 </signal>
 <signal name="REXT">
@@
 <contactref element="LED4" pad="C"/>
 <contactref element="R5" pad="2"/>
-<wire x1="3.8268" y1="32.9184" x2="2.4416" y2="31.5332" width="0.2032" layer="1"/>
-<wire x1="2.4416" y1="31.5332" x2="2.4384" y2="31.5332" width="0.2032" layer="1"/>
+<wire x1="5.4896" y1="31.9396" x2="6.4684" y2="32.9184" width="0.2032" layer="1"/>
+<wire x1="2.4384" y1="31.9396" x2="5.4896" y2="31.9396" width="0.2032" layer="1"/>
 </signal>
 <signal name="N$10">
@@
 </signal>
 </signals>
+<errors>
+</errors>
 </board>
 </drawing>

Commit message: value update
Parts:
- C29, C30: value 16p -> 18p
- R36: value 120 -> 100k
Changed lines of the file:
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@@
 <element name="U5" library="balto" package="SO08" value="MAX3051" x="31.496" y="5.08" rot="MR180"/>
 <element name="R35" library="rcl" package="R0805" value="120" x="24.9936" y="13.8176" rot="MR90"/>
-<element name="R36" library="rcl" package="R0603" value="120" x="27.432" y="1.8288" rot="MR0"/>
+<element name="R36" library="rcl" package="R0603" value="100k" x="27.432" y="1.8288" rot="MR0"/>
 <element name="C34" library="rcl" package="C0603" value="100n" x="34.544" y="6.2992" rot="MR90"/>
 <element name="R16" library="rcl" package="R0805" value="75" x="36.7792" y="10.5664" rot="MR90"/>
@@
 <element name="C8" library="rcl" package="C0603" value=".1u" x="41.8592" y="4.064" rot="MR225"/>
 <element name="U4" library="SparkFun-PowerIC" package="SOT23-5" value="MIC5301" x="41.656" y="8.128" rot="MR180"/>
-<element name="C29" library="rcl" package="C0603" value="16p" x="42.672" y="31.2928" rot="MR270"/>
-<element name="C30" library="rcl" package="C0603" value="16p" x="39.8272" y="31.2928" rot="MR90"/>
+<element name="C29" library="rcl" package="C0603" value="18p" x="42.672" y="31.2928" rot="MR270"/>
+<element name="C30" library="rcl" package="C0603" value="18p" x="39.8272" y="31.2928" rot="MR90"/>
 <element name="C6" library="rcl" package="C0603" value=".1u" x="30.8864" y="26.0096" rot="R180"/>
 <element name="C17" library="rcl" package="C0603" value=".1u" x="36.9824" y="31.496" rot="R90"/>
@@
 </signal>
 </signals>
-<errors>
-</errors>
 </board>
 </drawing>

Commit message: add silk and gnd vias
Routing:
- net GND: vias 19 -> 44
Other:
- board text added: "FB2013"
- board text added: "nrf-ethernet"
- board text added: "rev0"
Changed lines of the file:
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@@
 <layer number="27" name="tValues" color="7" fill="1" visible="no" active="yes"/>
 <layer number="28" name="bValues" color="7" fill="1" visible="no" active="yes"/>
-<layer number="29" name="tStop" color="7" fill="3" visible="no" active="yes"/>
-<layer number="30" name="bStop" color="7" fill="6" visible="no" active="yes"/>
+<layer number="29" name="tStop" color="7" fill="3" visible="yes" active="yes"/>
+<layer number="30" name="bStop" color="7" fill="6" visible="yes" active="yes"/>
 <layer number="31" name="tCream" color="7" fill="4" visible="no" active="yes"/>
 <layer number="32" name="bCream" color="7" fill="5" visible="no" active="yes"/>
@@
 <dimension x1="6.2992" y1="0" x2="53.4416" y2="-3.048" x3="-2.4384" y3="-1.524" textsize="1.778" layer="20" dtype="vertical"/>
 <rectangle x1="54.2544" y1="15.0368" x2="55.88" y2="16.6624" layer="29"/>
+<text x="68.2752" y="15.0368" size="1.778" layer="121" rot="SR270">FB2013</text>
+<text x="67.056" y="15.0368" size="1.016" layer="121" rot="SR270">nrf-ethernet</text>
+<text x="67.056" y="3.8608" size="1.016" layer="121" rot="SR270">rev0</text>
 </plain>
 <attributes>
@@
 <wire x1="37.7952" y1="33.3248" x2="44.704" y2="33.3248" width="0.2032" layer="1"/>
 <wire x1="44.704" y1="33.3248" x2="37.7952" y2="33.3248" width="0.2032" layer="16"/>
+<via x="66.04" y="13.4112" extent="1-16" drill="0.508"/>
+<via x="66.04" y="11.7856" extent="1-16" drill="0.508"/>
+<via x="66.04" y="10.16" extent="1-16" drill="0.508"/>
+<via x="66.04" y="8.5344" extent="1-16" drill="0.508"/>
+<via x="66.04" y="6.9088" extent="1-16" drill="0.508"/>
+<via x="66.04" y="5.2832" extent="1-16" drill="0.508"/>
+<via x="66.04" y="3.6576" extent="1-16" drill="0.508"/>
+<via x="66.04" y="2.032" extent="1-16" drill="0.508"/>
+<via x="66.04" y="18.8976" extent="1-16" drill="0.508"/>
+<via x="66.04" y="20.5232" extent="1-16" drill="0.508"/>
+<via x="66.04" y="22.1488" extent="1-16" drill="0.508"/>
+<via x="66.04" y="23.7744" extent="1-16" drill="0.508"/>
+<via x="66.04" y="25.4" extent="1-16" drill="0.508"/>
+<via x="66.04" y="27.0256" extent="1-16" drill="0.508"/>
+<via x="66.04" y="28.6512" extent="1-16" drill="0.508"/>
+<via x="66.04" y="30.2768" extent="1-16" drill="0.508"/>
+<via x="66.04" y="31.9024" extent="1-16" drill="0.508"/>
+<via x="63.6016" y="12.8016" extent="1-16" drill="0.508"/>
+<via x="63.6016" y="11.5824" extent="1-16" drill="0.508"/>
+<via x="58.3184" y="22.352" extent="1-16" drill="0.508"/>
+<via x="56.896" y="22.1488" extent="1-16" drill="0.508"/>
+<via x="59.7408" y="20.9296" extent="1-16" drill="0.508"/>
+<via x="1.6256" y="21.9456" extent="1-16" drill="0.508"/>
+<via x="19.1008" y="22.5552" extent="1-16" drill="0.508"/>
+<via x="34.544" y="8.5344" extent="1-16" drill="0.508"/>
 </signal>
 <signal name="TX+">
@@
 </signal>
 </signals>
+<errors>
+</errors>
 </board>
 </drawing>
